File: hardware/RP2350_60QFN_minimal.kicad_sch (KiCad schematic)
At the start: 43 parts, among them J1 USB_B_Micro, J2 Conn_02x18_Odd_Even, J3 Conn_02x18_Odd_Even, J4 SM03B-SRSS-TB, SW1 SW_Push, SW2 SW_Push, U1 RP2350_60QFN, U2 NCP1117-3.3_SOT223, U3 W25Q128JVS, Y1 ABM8-272-T3

Commit message: commit
Other:
- added sheet analog frontend (analog.kicad_sch)
